Commit message: cad: D047 — leg chain rebuilt around the real ST3215 (STEP-measured); review, print plan, shopping list; repo hygiene
Review (docs/REVIEW_2026-09-22.md): the v0.1 servo model was a guessed box
wrong in five ways (28.8 not 32 tall, horn top 33.1 not 38, axis 10.2 not
11.25 from the front, 45-degree hole pattern, no rear idler/rims/connectors),
so every D046 leg part was designed for a servo that does not exist and the
D046 yaw bearing stage would have failed. Servo v2 is derived from
cad/ref/STS3215_03a.step (SO-ARM100, Apache-2.0) with a self-check against
it; every number is in params.yaml marked "from STEP".

D047 leg: yaw servo shaft-down in a cup on the I1 base; one C-shaped fork
riding the horn below and the rear idler above; twin-plate femur (plate A on
the couplers, plate B on the idlers); knee cup on the tibia; servo_cup = one
retention shape for all three servos (four self-tappers into the rim holes);
coupler re-cut (lobes 0/90/180/270, slotted M3/M2 holes); blank v0.3 + glue-on
idler; four joint coupons. Hip axis 61 = params.leg.hip_axis_z, read by gait,
MJCF and URDF. check_assembly gains plug keep-outs, slot-end driver access,
rim-screw access and hip/knee sweeps. CAD CI 23/23 tree clean; mass 2665 g;
sim walk unchanged (264 mm, 1 deg); 85 fast tests; URDF parity restored
(masses from mass_budget.json, built-in macro expander).

Docs: PRINT_PLAN_2026-09-22 (coupons -> one leg -> body),
bom/SHOPPING_LIST_2026-09-22 (bench kit, full robot), D047, B22-B28,
BUILD_LOG session 9, README status. Repo: MIT LICENSE, .mcp.json untracked,
duplicates + NEXT_SESSION.md + stale exports removed, jpg/pdf on LFS,
first-prints photo filed under media/.

Co-Authored-By: Claude Fable 5.1 <noreply@anthropic.com>
Claude-Session: https://claude.ai/code/session_0147dyVvKxLRmCvJjDwaBeif

File: rocky_v0.8.0_code/rocky/ros2/rocky_description/urdf/pebble.urdf (robot description, URDF)
Before this commit: robot pebble, 26 links, 25 joints
Links:
- link base_link: mass 1.35 -> 1.4489
- link coxa0: mass 0.14 -> 0.0783
- link coxa1: mass 0.14 -> 0.0783
- link coxa2: mass 0.14 -> 0.0783
- link coxa3: mass 0.14 -> 0.0783
- link coxa4: mass 0.14 -> 0.0783
- link femur0: mass 0.03 -> 0.034
- link femur1: mass 0.03 -> 0.034
- link femur2: mass 0.03 -> 0.034
- link femur3: mass 0.03 -> 0.034
- link femur4: mass 0.03 -> 0.034
- link foot0: mass 0.05500000000000001 -> 0.043300000000000005
- link foot1: mass 0.05500000000000001 -> 0.043300000000000005
- link foot2: mass 0.05500000000000001 -> 0.043300000000000005
- link foot3: mass 0.05500000000000001 -> 0.043300000000000005
- link foot4: mass 0.05500000000000001 -> 0.043300000000000005
- link tibia0: mass 0.119 -> 0.0917
- link tibia1: mass 0.119 -> 0.0917
- link tibia2: mass 0.119 -> 0.0917
- link tibia3: mass 0.119 -> 0.0917
- link tibia4: mass 0.119 -> 0.0917
Joints:
- joint hip0: origin xyz=0.0450 0 0.0580 -> xyz=0.0450 0 0.0610
- joint hip1: origin xyz=0.0450 0 0.0580 -> xyz=0.0450 0 0.0610
- joint hip2: origin xyz=0.0450 0 0.0580 -> xyz=0.0450 0 0.0610
- joint hip3: origin xyz=0.0450 0 0.0580 -> xyz=0.0450 0 0.0610
- joint hip4: origin xyz=0.0450 0 0.0580 -> xyz=0.0450 0 0.0610

File: rocky_v0.8.0_code/rocky/ros2/rocky_description/urdf/pebble.urdf.xacro (robot description, xacro)
@@ -4,5 +4,5 @@
   <material name="pebble"><color rgba="0.55 0.42 0.75 1"/></material>
   <link name="base_link">
-    <inertial><origin xyz="0.000000 0.000000 0.024500"/><mass value="1.35"/><inertia ixx="3.805e-03" ixy="0" ixz="0" iyy="3.805e-03" iyz="0" izz="7.126e-03"/></inertial>
+    <inertial><origin xyz="0.000000 0.000000 0.024500"/><mass value="1.4489"/><inertia ixx="4.084e-03" ixy="0" ixz="0" iyy="4.084e-03" iyz="0" izz="7.648e-03"/></inertial>
     <visual><origin xyz="0 0 0.018"/>
       <geometry><cylinder radius="0.1100" length="0.024"/></geometry>
@@ -18,5 +18,5 @@
   <xacro:macro name="pebble_leg" params="i angle">
     <link name="coxa${i}">
-      <inertial><origin xyz="0.020000 0.000000 0.030000"/><mass value="0.14"/><inertia ixx="5.395e-05" ixy="0" ixz="0" iyy="8.400e-05" iyz="0" izz="5.395e-05"/></inertial>
+      <inertial><origin xyz="0.020000 0.000000 0.030000"/><mass value="0.0783"/><inertia ixx="3.017e-05" ixy="0" ixz="0" iyy="4.698e-05" iyz="0" izz="3.017e-05"/></inertial>
       <visual><origin xyz="0.020 0 0.030"/>
         <geometry><box size="0.060 0.032 0.060"/></geometry>
@@ -35,5 +35,5 @@
     </joint>
     <link name="femur${i}">
-      <inertial><origin xyz="0.047500 0.000000 0.000000"/><mass value="0.03"/><inertia ixx="2.160e-06" ixy="0" ixz="0" iyy="2.364e-05" iyz="0" izz="2.364e-05"/></inertial>
+      <inertial><origin xyz="0.047500 0.000000 0.000000"/><mass value="0.034"/><inertia ixx="2.448e-06" ixy="0" ixz="0" iyy="2.679e-05" iyz="0" izz="2.679e-05"/></inertial>
       <visual><origin xyz="0.0475 0 0" rpy="0 1.570796 0"/>
         <geometry><cylinder radius="0.012" length="0.0950"/></geometry>
@@ -44,5 +44,5 @@
     <joint name="hip${i}" type="revolute">
       <parent link="coxa${i}"/><child link="femur${i}"/>
-      <origin xyz="0.0450 0 0.0580"/>
+      <origin xyz="0.0450 0 0.0610"/>
       <axis xyz="0 -1 0"/>
       <limit lower="-1.221730" upper="1.570796"
@@ -51,5 +51,5 @@
     </joint>
     <link name="tibia${i}">
-      <inertial><origin xyz="0.062100 0.000000 0.000000"/><mass value="0.119"/><inertia ixx="5.950e-06" ixy="0" ixz="0" iyy="1.559e-04" iyz="0" izz="1.559e-04"/></inertial>
+      <inertial><origin xyz="0.062100 0.000000 0.000000"/><mass value="0.0917"/><inertia ixx="4.585e-06" ixy="0" ixz="0" iyy="1.202e-04" iyz="0" izz="1.202e-04"/></inertial>
       <visual><origin xyz="0.0621 0 0" rpy="0 1.570796 0"/>
         <geometry><cylinder radius="0.010" length="0.1242"/></geometry>
@@ -67,5 +67,5 @@
     </joint>
     <link name="foot${i}">
-      <inertial><origin xyz="0.000000 0.000000 0.000000"/><mass value="0.05500000000000001"/><inertia ixx="3.448e-06" ixy="0" ixz="0" iyy="3.448e-06" iyz="0" izz="3.448e-06"/></inertial>  <!-- +0.004: fixed claw prong (MJCF parity) -->
+      <inertial><origin xyz="0.000000 0.000000 0.000000"/><mass value="0.043300000000000005"/><inertia ixx="2.657e-06" ixy="0" ixz="0" iyy="2.657e-06" iyz="0" izz="2.657e-06"/></inertial>  <!-- +0.004: fixed claw prong (MJCF parity) -->
       <visual><geometry><sphere radius="0.013"/></geometry>
         <material name="pebble"/></visual>
