Commit message: D052: the sim stops flattering the servo; the studio cannot author what the robot cannot do; the bus gets a safe first move
Full review round (4 expert reviewers + 29 adversarially verified findings + a
three-lens review of the diff), then eight implementation packages:

- one servo identity: params.yaml actuators/joints/gait/reflex/sensing blocks
  read by gait/rocky_model.py; MJCF, URDF, servo_model, shove, driver clamp,
  playground and cockpit all read it (old keys are YAML aliases, not copies)
- physics: joint damping = stall/no-load (the DC torque-speed line, 0.626),
  leg forcerange = 0.65 x stall (continuous), foot mu 0.8 + torsional, foot
  sphere surface = IK foot point, claw double-count removed, world geoms get
  priority=1 so world friction reaches the feet, robot-only model fingerprint
- gait envelope: T 2.0 s / step 24 mm; WaveGait.budget() scales every command
  source into 45.5 mm/s and 0.246 rad/s; gait presets as data (gait/gaits/)
- one feasibility checker (gait/pebble_feasibility.py: limits with a guard
  band, speed per class loaded 3.0 / free 4.0 / hard 4.7, jumps, >=3 feet,
  CoM margin, slip, self-contact) gating code gestures, keyframe files, the
  studio, presets and the brain's compose_gesture; reach keyframes, a
  whole-body reach solver and teach-by-demonstration (gait/pebble_pose_solver.py);
  fist_bump re-authored in joint space, beckon/turn/claw/shake slowed to budget
- always-on loop: gestures blend in/out with the reflex still watching, one
  void guard for every command source (latched bearing, `clear`), 3 trips in
  5 s latch a safe stop, lead-limited contact probe, kinematic height, sim IMU
  from model gravity, servo model on by default, NaN-hold + 4.7 rad/s clamp
  before the sim and the bus
- RL on the robot's own path and sensors: obs v2 (EMA action, servo model in
  the loop, IMU/encoder/foot-switch noise, no torso height), rim shoves in the
  gait env, shared DR (voltage-correlated torque/speed, kp, CoM offset, joint
  offsets), SAME_STEP autoreset, env contract + fingerprint in checkpoints,
  seeded evals, --randomize and --supervisor columns, handoff_ok shared with
  the reflex supervisor
- hardware bridge made safe before any servo touched it: soft entry (park at
  the real pose, torque 40 %, 200 c/s, blend), refuse sim2real unless idle,
  locomotion held until real contacts exist, tolerant sync reads, per-leg
  fault cuts, degraded/lost/stale/nan events, heartbeat, jog in the gait
  frame, calibration re-derivation, apply_limits (EEPROM angle limits),
  per-tick rate limit at the bus, stream at the 50 Hz bus rate
- cockpit: sim thread failure fails every pending call and limps the bridge,
  tool args validated, chat history bounded and locked, model roles
  (brain / vision / multimodal / stt) with fallback chains and timeouts,
  vision detection from llama-swap descriptions, enable_thinking off, voice
  junk filter + wake word for motion, intent fixes (turn left/right, number
  words, look), goto reactive layer with a 'blocked' outcome, --unsafe-lan +
  Origin/Content-Type middleware, studio feasibility readout / reach / solve /
  teach UI, hardware panel wiring, gait presets, void/latch chips
- launcher/CI: train-walk fixed (--env gait), help prints everything, test
  ladder = CI, run_sim exits non-zero on a fall or a displacement outside the
  band, generated files checked for staleness, cad job on PRs touching cad/
- bugs found on the way: CockpitBackend gesture over MCP always failed
  (argument-name collision), rl_dashboard/run_sim numbers stale
- measured on the new model: run_sim 246 mm of 261, tilt 0.84 deg max; standing
  survives 30-35 N rim shoves (was 25); recover1 is 2/20 legacy / 0/20 hardware
  handoff (was 7/20) while the supervisor system number is 20/20 with the
  righter vs 11/20 without; all shipped gestures pass the audit (0 FAIL)
- NOT verified: any real servo; tailnet; a righter retrained on obs v2 (B34)
- open decision recorded as a strict xfail: forcerange = continuous torque caps
  a free joint at 3.06 rad/s below the 4.0 free budget (peak torque + thermal
  limit is the likely fix)

Co-Authored-By: Claude Fable 5.1 <noreply@anthropic.com>
Claude-Session: https://claude.ai/code/session_0147dyVvKxLRmCvJjDwaBeif

File: ros2/rocky_description/urdf/pebble.urdf (robot description, URDF)
Before this commit: robot pebble, 26 links, 25 joints
Links:
- link femur0: mass 0.034 -> 0.035
- link femur1: mass 0.034 -> 0.035
- link femur2: mass 0.034 -> 0.035
- link femur3: mass 0.034 -> 0.035
- link femur4: mass 0.034 -> 0.035
- link foot0: geometry collision sphere radius=0.0065; visual cylinder length=0.028 radius=0.0035
- link foot1: geometry collision sphere radius=0.0065; visual cylinder length=0.028 radius=0.0035
- link foot2: geometry collision sphere radius=0.0065; visual cylinder length=0.028 radius=0.0035
- link foot3: geometry collision sphere radius=0.0065; visual cylinder length=0.028 radius=0.0035
- link foot4: geometry collision sphere radius=0.0065; visual cylinder length=0.028 radius=0.0035
- link tibia0: mass 0.0917 -> 0.0837
- link tibia1: mass 0.0917 -> 0.0837
- link tibia2: mass 0.0917 -> 0.0837
- link tibia3: mass 0.0917 -> 0.0837
- link tibia4: mass 0.0917 -> 0.0837
Joints:
- joint claw0: limit lower=0.000000 upper=0.959931 effort=0.23 velocity=6.0 -> lower=0.000000 upper=0.959931 effort=0.1495 velocity=9.5
- joint claw1: limit lower=0.000000 upper=0.959931 effort=0.23 velocity=6.0 -> lower=0.000000 upper=0.959931 effort=0.1495 velocity=9.5
- joint claw2: limit lower=0.000000 upper=0.959931 effort=0.23 velocity=6.0 -> lower=0.000000 upper=0.959931 effort=0.1495 velocity=9.5
- joint claw3: limit lower=0.000000 upper=0.959931 effort=0.23 velocity=6.0 -> lower=0.000000 upper=0.959931 effort=0.1495 velocity=9.5
- joint claw4: limit lower=0.000000 upper=0.959931 effort=0.23 velocity=6.0 -> lower=0.000000 upper=0.959931 effort=0.1495 velocity=9.5
- joint hip0: limit lower=-1.221730 upper=1.570796 effort=2.94 velocity=5.2 -> lower=-1.221730 upper=1.570796 effort=1.9110 velocity=4.7
- joint hip1: limit lower=-1.221730 upper=1.570796 effort=2.94 velocity=5.2 -> lower=-1.221730 upper=1.570796 effort=1.9110 velocity=4.7
- joint hip2: limit lower=-1.221730 upper=1.570796 effort=2.94 velocity=5.2 -> lower=-1.221730 upper=1.570796 effort=1.9110 velocity=4.7
- joint hip3: limit lower=-1.221730 upper=1.570796 effort=2.94 velocity=5.2 -> lower=-1.221730 upper=1.570796 effort=1.9110 velocity=4.7
- joint hip4: limit lower=-1.221730 upper=1.570796 effort=2.94 velocity=5.2 -> lower=-1.221730 upper=1.570796 effort=1.9110 velocity=4.7
- joint knee0: limit lower=-2.617994 upper=-0.349066 effort=2.94 velocity=5.2 -> lower=-2.617994 upper=-0.349066 effort=1.9110 velocity=4.7
- joint knee1: limit lower=-2.617994 upper=-0.349066 effort=2.94 velocity=5.2 -> lower=-2.617994 upper=-0.349066 effort=1.9110 velocity=4.7
- joint knee2: limit lower=-2.617994 upper=-0.349066 effort=2.94 velocity=5.2 -> lower=-2.617994 upper=-0.349066 effort=1.9110 velocity=4.7
- joint knee3: limit lower=-2.617994 upper=-0.349066 effort=2.94 velocity=5.2 -> lower=-2.617994 upper=-0.349066 effort=1.9110 velocity=4.7
- joint knee4: limit lower=-2.617994 upper=-0.349066 effort=2.94 velocity=5.2 -> lower=-2.617994 upper=-0.349066 effort=1.9110 velocity=4.7
- joint yaw0: limit lower=-0.698132 upper=0.698132 effort=2.94 velocity=5.2 -> lower=-0.698132 upper=0.698132 effort=1.9110 velocity=4.7
- joint yaw1: limit lower=-0.698132 upper=0.698132 effort=2.94 velocity=5.2 -> lower=-0.698132 upper=0.698132 effort=1.9110 velocity=4.7
- joint yaw2: limit lower=-0.698132 upper=0.698132 effort=2.94 velocity=5.2 -> lower=-0.698132 upper=0.698132 effort=1.9110 velocity=4.7
- joint yaw3: limit lower=-0.698132 upper=0.698132 effort=2.94 velocity=5.2 -> lower=-0.698132 upper=0.698132 effort=1.9110 velocity=4.7
- joint yaw4: limit lower=-0.698132 upper=0.698132 effort=2.94 velocity=5.2 -> lower=-0.698132 upper=0.698132 effort=1.9110 velocity=4.7

File: ros2/rocky_description/urdf/pebble.urdf.xacro (robot description, xacro)
@@ -31,9 +31,9 @@
       <axis xyz="0 0 1"/>
       <limit lower="-0.698132" upper="0.698132"
-             effort="2.94" velocity="5.2"/>
-      <dynamics damping="0.05"/>
+             effort="1.9110" velocity="4.7"/>
+      <dynamics damping="0.6255"/>
     </joint>
     <link name="femur${i}">
-      <inertial><origin xyz="0.047500 0.000000 0.000000"/><mass value="0.034"/><inertia ixx="2.448e-06" ixy="0" ixz="0" iyy="2.679e-05" iyz="0" izz="2.679e-05"/></inertial>
+      <inertial><origin xyz="0.047500 0.000000 0.000000"/><mass value="0.035"/><inertia ixx="2.520e-06" ixy="0" ixz="0" iyy="2.758e-05" iyz="0" izz="2.758e-05"/></inertial>
       <visual><origin xyz="0.0475 0 0" rpy="0 1.570796 0"/>
         <geometry><cylinder radius="0.012" length="0.0950"/></geometry>
@@ -47,9 +47,9 @@
       <axis xyz="0 -1 0"/>
       <limit lower="-1.221730" upper="1.570796"
-             effort="2.94" velocity="5.2"/>
-      <dynamics damping="0.05"/>
+             effort="1.9110" velocity="4.7"/>
+      <dynamics damping="0.6255"/>
     </joint>
     <link name="tibia${i}">
-      <inertial><origin xyz="0.062100 0.000000 0.000000"/><mass value="0.0917"/><inertia ixx="4.585e-06" ixy="0" ixz="0" iyy="1.202e-04" iyz="0" izz="1.202e-04"/></inertial>
+      <inertial><origin xyz="0.062100 0.000000 0.000000"/><mass value="0.0837"/><inertia ixx="4.185e-06" ixy="0" ixz="0" iyy="1.097e-04" iyz="0" izz="1.097e-04"/></inertial>
       <visual><origin xyz="0.0621 0 0" rpy="0 1.570796 0"/>
         <geometry><cylinder radius="0.010" length="0.1242"/></geometry>
@@ -63,15 +63,15 @@
       <axis xyz="0 -1 0"/>
       <limit lower="-2.617994" upper="-0.349066"
-             effort="2.94" velocity="5.2"/>
-      <dynamics damping="0.05"/>
+             effort="1.9110" velocity="4.7"/>
+      <dynamics damping="0.6255"/>
     </joint>
     <link name="foot${i}">
-      <inertial><origin xyz="0.000000 0.000000 0.000000"/><mass value="0.043300000000000005"/><inertia ixx="2.657e-06" ixy="0" ixz="0" iyy="2.657e-06" iyz="0" izz="2.657e-06"/></inertial>  <!-- +0.004: fixed claw prong (MJCF parity) -->
-      <visual><geometry><sphere radius="0.013"/></geometry>
+      <inertial><origin xyz="-0.006500 0.000000 0.000000"/><mass value="0.043300000000000005"/><inertia ixx="6.642e-07" ixy="0" ixz="0" iyy="6.642e-07" iyz="0" izz="6.642e-07"/></inertial>  <!-- + fixed claw prong (MJCF parity) -->
+      <visual><origin xyz="-0.0065 0 0"/><geometry><sphere radius="0.0065"/></geometry>
         <material name="pebble"/></visual>
       <visual><origin xyz="0.012 0.0075 0" rpy="0 0 0.28"/>
         <geometry><cylinder radius="0.0035" length="0.028"/></geometry>
         <material name="pebble"/></visual>
-      <collision><geometry><sphere radius="0.013"/></geometry></collision>
+      <collision><origin xyz="-0.0065 0 0"/><geometry><sphere radius="0.0065"/></geometry></collision>
     </link>
     <joint name="foot_fix${i}" type="fixed">
@@ -90,5 +90,5 @@
       <axis xyz="0 0 1"/>
       <limit lower="0.000000" upper="0.959931"
-             effort="0.23" velocity="6.0"/>
+             effort="0.1495" velocity="9.5"/>
       <dynamics damping="0.01"/>
     </joint>

Commit message: D052a: peak torque with a thermal budget, the shallow-angle cliff miss, spawn-pose bug, leftovers
- physics: leg forcerange = stall (2.94 N.m, instantaneous) — the 0.65 x stall
  clip was wrong as an instantaneous cap: it held an unloaded joint at 3.06
  rad/s, below the servo's 4.7 no-load speed and the 4.0 free-leg budget.
  Damping unchanged (the DC line: 4.7 at zero load, 3.05 at continuous torque).
  The continuous budget is now a THERMAL model over time: rl_common.ThermalProxy
  in both RL envs (electrical torque, integrator matched to the driver mock's
  thermal curve: trips after 180 s at 0.85 x stall, 94 s at stall; derate ramps
  to continuous + a reward penalty), a THERMAL_LOAD verdict in the feasibility
  checker (RMS load), a load column in audit_gestures, a servo-heat chip in the
  cockpit and sim2real refused past the budget. URDF effort = peak, velocity =
  no-load, parity checks both. The strict xfail is gone.
- void guard at 10-20 deg approaches: the wave gait lifts the next leg exactly
  when the previous lands, so two leading legs straddle the edge and the CoM
  leaves the remaining triangle in ~0.3 s. Fix: a touchdown gate (the gait clock
  waits until the landing foot reports contact or its probe exhausts) and a
  retreat that plays the approach backwards; optional careful walk (gate.wait,
  off: -17 % speed). Stop margins at walk 45: 0/10/15/20/30/45 deg all stop
  (was falls at 10, 15, 20); 72-approach sweep 28 falls -> 6 (lip footholds,
  pinned as a strict xfail, B33 candidate); no false voids on rubble/rough/stairs.
- an older bug: four scripts wrote the leg angles into qpos[7:22] although the
  claw joints interleave — every push/terrain trial spawned 9.8 deg tilted and
  reported that as its tilt max. Fixed in run_sim, run_push, run_push_reflex,
  run_terrain, run_sim_manip, audit_righter and the model test.
- leftovers: ppo_smoke obs_dim from the env, spawn height from rocky_model in
  every script, GOTO_DOC 'blocked' meaning, UI sim2real gate (idle + speed 1x),
  set_world resets yaw on a different world, SIM_GUIDE 2/5, RL_GUIDE 1, README
  counts, decisions D052 amended + D052a row, BUILD_LOG addendum.
- re-measured: run_sim 246 mm / 0.84 deg unchanged; standing shove floor 29 N
  (1.11 BW) on a 1 N grid, 2 N lower than with the continuous clip (stiffer
  knees pivot instead of sliding); righter under the supervisor still 20/20
  vs 11/20, stands faster (0.46 s vs 0.80 s); recover1 legacy handoff 5/20
  (20-episode noise around 2-3/20), hardware handoff 0/20.
- fast suite 325 passed, 2 xfailed (both strict, both documented gaps).

Co-Authored-By: Claude Fable 5.1 <noreply@anthropic.com>
Claude-Session: https://claude.ai/code/session_0147dyVvKxLRmCvJjDwaBeif

File: ros2/rocky_description/urdf/pebble.urdf (robot description, URDF)
Before this commit: robot pebble, 26 links, 25 joints
Joints:
- joint claw0: limit lower=0.000000 upper=0.959931 effort=0.1495 velocity=9.5 -> lower=0.000000 upper=0.959931 effort=0.2300 velocity=9.5
- joint claw1: limit lower=0.000000 upper=0.959931 effort=0.1495 velocity=9.5 -> lower=0.000000 upper=0.959931 effort=0.2300 velocity=9.5
- joint claw2: limit lower=0.000000 upper=0.959931 effort=0.1495 velocity=9.5 -> lower=0.000000 upper=0.959931 effort=0.2300 velocity=9.5
- joint claw3: limit lower=0.000000 upper=0.959931 effort=0.1495 velocity=9.5 -> lower=0.000000 upper=0.959931 effort=0.2300 velocity=9.5
- joint claw4: limit lower=0.000000 upper=0.959931 effort=0.1495 velocity=9.5 -> lower=0.000000 upper=0.959931 effort=0.2300 velocity=9.5
- joint hip0: limit lower=-1.221730 upper=1.570796 effort=1.9110 velocity=4.7 -> lower=-1.221730 upper=1.570796 effort=2.9400 velocity=4.7
- joint hip1: limit lower=-1.221730 upper=1.570796 effort=1.9110 velocity=4.7 -> lower=-1.221730 upper=1.570796 effort=2.9400 velocity=4.7
- joint hip2: limit lower=-1.221730 upper=1.570796 effort=1.9110 velocity=4.7 -> lower=-1.221730 upper=1.570796 effort=2.9400 velocity=4.7
- joint hip3: limit lower=-1.221730 upper=1.570796 effort=1.9110 velocity=4.7 -> lower=-1.221730 upper=1.570796 effort=2.9400 velocity=4.7
- joint hip4: limit lower=-1.221730 upper=1.570796 effort=1.9110 velocity=4.7 -> lower=-1.221730 upper=1.570796 effort=2.9400 velocity=4.7
- joint knee0: limit lower=-2.617994 upper=-0.349066 effort=1.9110 velocity=4.7 -> lower=-2.617994 upper=-0.349066 effort=2.9400 velocity=4.7
- joint knee1: limit lower=-2.617994 upper=-0.349066 effort=1.9110 velocity=4.7 -> lower=-2.617994 upper=-0.349066 effort=2.9400 velocity=4.7
- joint knee2: limit lower=-2.617994 upper=-0.349066 effort=1.9110 velocity=4.7 -> lower=-2.617994 upper=-0.349066 effort=2.9400 velocity=4.7
- joint knee3: limit lower=-2.617994 upper=-0.349066 effort=1.9110 velocity=4.7 -> lower=-2.617994 upper=-0.349066 effort=2.9400 velocity=4.7
- joint knee4: limit lower=-2.617994 upper=-0.349066 effort=1.9110 velocity=4.7 -> lower=-2.617994 upper=-0.349066 effort=2.9400 velocity=4.7
- joint yaw0: limit lower=-0.698132 upper=0.698132 effort=1.9110 velocity=4.7 -> lower=-0.698132 upper=0.698132 effort=2.9400 velocity=4.7
- joint yaw1: limit lower=-0.698132 upper=0.698132 effort=1.9110 velocity=4.7 -> lower=-0.698132 upper=0.698132 effort=2.9400 velocity=4.7
- joint yaw2: limit lower=-0.698132 upper=0.698132 effort=1.9110 velocity=4.7 -> lower=-0.698132 upper=0.698132 effort=2.9400 velocity=4.7
- joint yaw3: limit lower=-0.698132 upper=0.698132 effort=1.9110 velocity=4.7 -> lower=-0.698132 upper=0.698132 effort=2.9400 velocity=4.7
- joint yaw4: limit lower=-0.698132 upper=0.698132 effort=1.9110 velocity=4.7 -> lower=-0.698132 upper=0.698132 effort=2.9400 velocity=4.7

File: ros2/rocky_description/urdf/pebble.urdf.xacro (robot description, xacro)
@@ -31,5 +31,5 @@
       <axis xyz="0 0 1"/>
       <limit lower="-0.698132" upper="0.698132"
-             effort="1.9110" velocity="4.7"/>
+             effort="2.9400" velocity="4.7"/>
       <dynamics damping="0.6255"/>
     </joint>
@@ -47,5 +47,5 @@
       <axis xyz="0 -1 0"/>
       <limit lower="-1.221730" upper="1.570796"
-             effort="1.9110" velocity="4.7"/>
+             effort="2.9400" velocity="4.7"/>
       <dynamics damping="0.6255"/>
     </joint>
@@ -63,5 +63,5 @@
       <axis xyz="0 -1 0"/>
       <limit lower="-2.617994" upper="-0.349066"
-             effort="1.9110" velocity="4.7"/>
+             effort="2.9400" velocity="4.7"/>
       <dynamics damping="0.6255"/>
     </joint>
@@ -90,6 +90,6 @@
       <axis xyz="0 0 1"/>
       <limit lower="0.000000" upper="0.959931"
-             effort="0.1495" velocity="9.5"/>
-      <dynamics damping="0.01"/>
+             effort="0.2300" velocity="9.5"/>
+      <dynamics damping="0.0242"/>
     </joint>
   </xacro:macro>

Commit message: cad: leg harness channel through coxa_yaw_base, star-board bracket on real deck holes, deterministic exports, 28 checks
- HWDOCS-01: the D047 base covered the deck's I1 pass-through; an 11 x 11 route now reaches the yaw plugs (6 checks)
- HWDOCS-02: bracket v0.2 bolts to grid holes (0,20)/(0,40) with a layout audit
- STEP write-if-changed + invariant PDF: regeneration no longer churns 57 STEPs
- run_all_checks 28 modules (+servo STEP comparison), --derived regenerates previews/estimate/print pack/viewer
- params: dead 683ZZ blocks out, bed_mm + xt60_panel_mm in; derived outputs regenerated (pre-D047 previews gone)
- torso 1448.9 -> 1435.2 g, robot fingerprint ceb63a1254c3 -> 7d376178fe27; 60 orphan renders removed
- print pack moved to cad/out/; Apache-2.0 text beside the servo STEP

Co-Authored-By: Claude Opus 5.5 (1M context) <noreply@anthropic.com>
Claude-Session: https://claude.ai/code/session_0147dyVvKxLRmCvJjDwaBeif

File: ros2/rocky_description/urdf/pebble.urdf (robot description, URDF)
Before this commit: robot pebble, 26 links, 25 joints
Links:
- link base_link: mass 1.4489 -> 1.4352

File: ros2/rocky_description/urdf/pebble.urdf.xacro (robot description, xacro)
@@ -4,5 +4,5 @@
   <material name="pebble"><color rgba="0.55 0.42 0.75 1"/></material>
   <link name="base_link">
-    <inertial><origin xyz="0.000000 0.000000 0.024500"/><mass value="1.4489"/><inertia ixx="4.084e-03" ixy="0" ixz="0" iyy="4.084e-03" iyz="0" izz="7.648e-03"/></inertial>
+    <inertial><origin xyz="0.000000 0.000000 0.024500"/><mass value="1.4352"/><inertia ixx="4.045e-03" ixy="0" ixz="0" iyy="4.045e-03" iyz="0" izz="7.576e-03"/></inertial>
     <visual><origin xyz="0 0 0.018"/>
       <geometry><cylinder radius="0.1100" length="0.024"/></geometry>

Commit message: D062: femur closed box (B74), sled fits its bay (B72), print pack rebuilt
- part_femur: plate B deck over the bridge + 8 mm rails; fem_check femur
  1.22 -> 2.18 (all five leg parts pass), knee deflection 4.5 -> 1.06 mm;
  the plate-B M3 holes no longer break out of the rails (new check), and
  take M3 x 12 (BOM A-18).
- battery sled: pack_w 46 -> 44 (sled 48.8 mm in the 50 mm bay); part_battery
  fails when sled + pack exceed the bay.
- params_rev D062, fingerprint 1f953c89f979, robot 2694.6 g; MJCF, URDF,
  mass budget, TOOLS.md regenerated; walk 247 mm, standing shove floor 30 N,
  knee self-right 50.3 %, recover1 system 20/20 unchanged; records updated.
- gen_print_pack: 44-page pack per batch in print order, print-pose views,
  strength verdicts, the TechDraw sheets merged (pypdf pinned), byte-stable.
- test_feasibility: MJCF summed-mass tolerance sized to its 0.1 g rounding.

Co-Authored-By: Claude Opus 5.5 (1M context) <noreply@anthropic.com>
Claude-Session: https://claude.ai/code/session_0147dyVvKxLRmCvJjDwaBeif

File: ros2/rocky_description/urdf/pebble.urdf (robot description, URDF)
Before this commit: robot pebble, 26 links, 25 joints
Links:
- link base_link: mass 1.4352 -> 1.4345999999999999
- link femur0: mass 0.035 -> 0.0427
- link femur1: mass 0.035 -> 0.0427
- link femur2: mass 0.035 -> 0.0427
- link femur3: mass 0.035 -> 0.0427
- link femur4: mass 0.035 -> 0.0427

File: ros2/rocky_description/urdf/pebble.urdf.xacro (robot description, xacro)
@@ -4,5 +4,5 @@
   <material name="pebble"><color rgba="0.55 0.42 0.75 1"/></material>
   <link name="base_link">
-    <inertial><origin xyz="0.000000 0.000000 0.024500"/><mass value="1.4352"/><inertia ixx="4.045e-03" ixy="0" ixz="0" iyy="4.045e-03" iyz="0" izz="7.576e-03"/></inertial>
+    <inertial><origin xyz="0.000000 0.000000 0.024500"/><mass value="1.4345999999999999"/><inertia ixx="4.043e-03" ixy="0" ixz="0" iyy="4.043e-03" iyz="0" izz="7.573e-03"/></inertial>
     <visual><origin xyz="0 0 0.018"/>
       <geometry><cylinder radius="0.1100" length="0.024"/></geometry>
@@ -35,5 +35,5 @@
     </joint>
     <link name="femur${i}">
-      <inertial><origin xyz="0.047500 0.000000 0.000000"/><mass value="0.035"/><inertia ixx="2.520e-06" ixy="0" ixz="0" iyy="2.758e-05" iyz="0" izz="2.758e-05"/></inertial>
+      <inertial><origin xyz="0.047500 0.000000 0.000000"/><mass value="0.0427"/><inertia ixx="3.074e-06" ixy="0" ixz="0" iyy="3.365e-05" iyz="0" izz="3.365e-05"/></inertial>
       <visual><origin xyz="0.0475 0 0" rpy="0 1.570796 0"/>
         <geometry><cylinder radius="0.012" length="0.0950"/></geometry>
