Commit message: D063: the leg is buildable, the shell latch works, smoother motion
CAD (the faults the assembly guide found, each implemented then
adversarially reviewed):
- B80/B81: the coxa fork slides onto the yaw servo and the blank (0 mm³ on
  the whole path; new check_assembly J1 path + seat checks). Opening the
  idler pocket lost the wall an inward foot push bears on (R- SF 0.49), so
  the fork gets side cheeks: SF 2.47 (governs), +5.5 g per fork. The horn
  face bears on a flat hub top.
- B82 knob keys an M3 x 16 hex head; B83 the I6 set screw clamps; B87 the I3
  latch assembles and bites (turned from below with a flat screwdriver);
  B88 hatch magnets seated; B89 Pi standoffs 58 x 49; B90 IMU pad fits the
  BNO085 and clears the Pi; B94 link_clip fits the D062 femur.

Motion (B76 fixes 1, 2, 3, 8; B79):
- soft-landing swing: lift-off/touchdown velocity step 3.05 -> 0 rad/s;
  the gait envelope 45.5 -> 34.2 mm/s (T 2.2 = 39.8 offered, not applied)
- command slew (rate limit + 0.2 s lag) wired into the supervisor, ROS
  node and playground; stops are never slewed; start 28.4 -> 3.4 deg/tick
- per-tick servo goal speed (k 1.3, VERIFY-ON-BENCH); minimum-jerk keyframe
  blends; register_dump reads 0-87
- the slew moved the cliff lip band: a faster hold probe keeps it at 8/364
  with 0 falls after a fired void guard; walking shove now at a steady
  envelope speed: 30 N (1.12 BW) every direction
- goto caps from the envelope (55 s, detour 15.5 s, go_back 300 s) and the
  3 s stuck rule now also runs during a detour

Model: fingerprint 1f953c89f979 -> 87215110e9c4, robot 2727.7 g,
params_rev D063; recover1 system 20/20; gestures 19 rows 0 FAIL.
Body interior (B51, B84-B86, B92, B93): docs/BODY_LAYOUT_PROPOSAL.md, owner
decisions pending. Follow-ups B97-B115. Tests: fast 1,078, slow 4 + 3
xfail, CAD 34/34 + FEM 5/5, byte-stable.

Co-Authored-By: Claude Opus 5.5 (1M context) <noreply@anthropic.com>
Claude-Session: https://claude.ai/code/session_0147dyVvKxLRmCvJjDwaBeif

File: ros2/rocky_description/urdf/pebble.urdf (robot description, URDF)
Before this commit: robot pebble, 26 links, 25 joints
Links:
- link base_link: mass 1.4345999999999999 -> 1.4397
- link coxa0: mass 0.0783 -> 0.0839
- link coxa1: mass 0.0783 -> 0.0839
- link coxa2: mass 0.0783 -> 0.0839
- link coxa3: mass 0.0783 -> 0.0839
- link coxa4: mass 0.0783 -> 0.0839

File: ros2/rocky_description/urdf/pebble.urdf.xacro (robot description, xacro)
@@ -4,5 +4,5 @@
   <material name="pebble"><color rgba="0.55 0.42 0.75 1"/></material>
   <link name="base_link">
-    <inertial><origin xyz="0.000000 0.000000 0.024500"/><mass value="1.4345999999999999"/><inertia ixx="4.043e-03" ixy="0" ixz="0" iyy="4.043e-03" iyz="0" izz="7.573e-03"/></inertial>
+    <inertial><origin xyz="0.000000 0.000000 0.024500"/><mass value="1.4397"/><inertia ixx="4.058e-03" ixy="0" ixz="0" iyy="4.058e-03" iyz="0" izz="7.600e-03"/></inertial>
     <visual><origin xyz="0 0 0.018"/>
       <geometry><cylinder radius="0.1100" length="0.024"/></geometry>
@@ -18,5 +18,5 @@
   <xacro:macro name="pebble_leg" params="i angle">
     <link name="coxa${i}">
-      <inertial><origin xyz="0.020000 0.000000 0.030000"/><mass value="0.0783"/><inertia ixx="3.017e-05" ixy="0" ixz="0" iyy="4.698e-05" iyz="0" izz="3.017e-05"/></inertial>
+      <inertial><origin xyz="0.020000 0.000000 0.030000"/><mass value="0.0839"/><inertia ixx="3.233e-05" ixy="0" ixz="0" iyy="5.034e-05" iyz="0" izz="3.233e-05"/></inertial>
       <visual><origin xyz="0.020 0 0.030"/>
         <geometry><box size="0.060 0.032 0.060"/></geometry>

Commit message: 9o: the 87 s detour goto cap (B116), torque audit counts the hands once (B106), CAD tidy (B105, B107, B108, B110)
- B116 (owner: "yes, apply the 87 s goto cap"): a goto that has entered a detour gets
  goto_cap_s with the reach grown by two detours (87 s at the 34.2 mm/s envelope) and ends at
  it even mid-detour (answers <= 88.5 s); a goto that never detoured keeps 55 s. go_back_to's
  proxy timeout is derived: 4 x (87 + 1.5) + 12 = 366 s. Verify on the shipped rule: 214/214
  as derived; around an obstacle 16/78/80/15 arrive at 1.0/1.2/1.5/2.0 m (55 s: 15/38/0/0).
- B106: the hands are inside the tibia link; the audit weighs the robot at 2727.8 g = the MJCF.
  Self-right knee 1.496 -> 1.397 N·m, 47.5 % of stall, HOT -> WARM.
- B110: one cad-check --derived --fem leaves a current print pack (FEM before the pack; the
  solver runs single-threaded). B105: drawings list open channels (the fork shows 3).
  B107: D-shaped latch housing, one way in. B108: the bus adapter, buck and UBEC get envelopes;
  they fit nowhere on the tray as drawn (an owner decision, with B51).
- Regenerated mass_budget / URDF (torso +0.1 g from B107; pebble.xml byte-identical).

Fingerprint unchanged (87215110e9c4). Fast ladder 1,101 passed; sim incl. slow 806 passed;
cad-check --derived 34/34, byte-stable over two passes.

Co-Authored-By: Claude Opus 5.5 (1M context) <noreply@anthropic.com>
Claude-Session: https://claude.ai/code/session_0147dyVvKxLRmCvJjDwaBeif

File: ros2/rocky_description/urdf/pebble.urdf (robot description, URDF)
Before this commit: robot pebble, 26 links, 25 joints
Links:
- link base_link: mass 1.4397 -> 1.4398

File: ros2/rocky_description/urdf/pebble.urdf.xacro (robot description, xacro)
@@ -4,5 +4,5 @@
   <material name="pebble"><color rgba="0.55 0.42 0.75 1"/></material>
   <link name="base_link">
-    <inertial><origin xyz="0.000000 0.000000 0.024500"/><mass value="1.4397"/><inertia ixx="4.058e-03" ixy="0" ixz="0" iyy="4.058e-03" iyz="0" izz="7.600e-03"/></inertial>
+    <inertial><origin xyz="0.000000 0.000000 0.024500"/><mass value="1.4398"/><inertia ixx="4.058e-03" ixy="0" ixz="0" iyy="4.058e-03" iyz="0" izz="7.600e-03"/></inertial>
     <visual><origin xyz="0 0 0.018"/>
       <geometry><cylinder radius="0.1100" length="0.024"/></geometry>

Commit message: D064 sim: the belly, the torso's real mass distribution, the righter's hip clamp (pick 13)
The sim never had a belly: its lowest torso surface was the cylinder at z +6
(124 mm over the ground) while option A's keel tub hangs to -55.4 (62.1 mm
settled), and the torso's mass sat on two cylinders at z 24.5. Pick 13 asks for
the belly in the sim plus a FALLEN/RIGHTED-only hip clamp on legs 1-4 (B97,
B130, B138, decision 13).

- gait/rocky_model.py: bay_tub_extent_mm() (the same sums as
  cad/iface.bay_tub_extent: x -97.5..101.9, y -47.4..7.4, z -55.4..-18.0 at
  bay_l 194), hub_shelf_extent_mm() (params x/y grown to the hull of the three
  Ø14 post pads: x -57..57, y 12.2..71, z -54.4..-10), belly_boxes(),
  righter_hip_min_deg() / righter_clamp_legs() (default 1-4), mass_budget() /
  torso_inertial().
- sim/mass_audit.py: a body-frame pose table for every torso item (STL
  centroids + mesh inertia where an STL exists, boxes otherwise; the 400 g
  pod split by location, every share VERIFY; the 380 g pack on the sled in the
  tub), writing torso_com_mm and the full torso_inertia; the retired parts are
  gone. --allow-missing (DEV ONLY) fills bay_tub / bay_door / bay_lid /
  hub_shelf with the proposal's masses and marks the budget provisional.
- sim/build_mjcf.py: the torso's explicit <inertial> from the budget, the two
  cylinders at mass 0, two massless contact boxes belly_tub / belly_shelf
  after <freejoint/>. URDF base_link carries the same inertial + boxes;
  check_urdf_parity compares the torso inertial.
- gait/pebble_reflex.py: the clamp in FALLEN (the righter's or the hold's
  command) and therefore on RIGHTED's ramp start; never in NORMAL / BRACE /
  RECOVER / probes (B129). rocky_recover_env maps legs 1-4's hip over
  [-51.05, 90] for new runs; old checkpoints replay their uncut map (contract
  key hip_floor_deg); PolicyRighter follows the contract.
- gait/pebble_feasibility.py: M_TORSO and TORSO_COM from the budget (B138);
  a leg in the belly is a SELF_CONTACT named belly_tub / belly_shelf.
- eval_recover / audit_righter report the FALLEN/RIGHTED hip-command minimum,
  the clamp's share of FALLEN ticks and every belly contact (box, leg, state).
  Smoke, recover1 + supervisor, 40 seeds (20 falls): clamp on 0 FALLEN/RIGHTED
  tub contacts, off 2 (leg 1, max 3.52 mm), stood 39/40 both, 41.3 % of FALLEN
  ticks clamped; leg 0 (not in the set) touches the shelf hull in 20/20 falls
  (max 2.93 mm, on the hull's north face at y 70-71, past the plate's 64.2).
- The lip-band approaches now tip onto the keel tub at the edge and fire the
  void 1.1-1.3 s later at 20-22 deg: the strict xfail counts that tip as a fall.
- Tests: test_belly.py (boxes vs params, inertial vs budget, DR bases, the
  remapped action range, the clamp through the real stack); the shove torque
  for an off-axis CoM; the contact-threshold lift follows the robot weight;
  the lip-band xfail counts a tip onto the keel as a fall; torque_audit reads
  only the gram keys.

PROVISIONAL: the four new parts have no STL in this tree, so the budget
(torso 1527.6 g at (-2.12, -3.95, -2.55) mm, robot 2815.6 g) and everything
generated from it (pebble.xml, URDF, urdf_parity.json, out/torque_audit.json)
must be regenerated at integration with mass_audit (no flag). Fingerprint
87215110e9c4 -> c10b970d2bb2 (provisional); every RL checkpoint is legacy.

Co-Authored-By: Claude Opus 5.5 <noreply@anthropic.com>
Claude-Session: https://claude.ai/code/session_01XWxNpsfCHorgwmudjicXmk

File: ros2/rocky_description/urdf/pebble.urdf (robot description, URDF)
Before this commit: robot pebble, 26 links, 25 joints
Links:
- link base_link: mass 1.4398 -> 1.5276; geometry collision box size=0.11400 0.05880 0.04440; collision box size=0.19940 0.05480 0.03740

File: ros2/rocky_description/urdf/pebble.urdf.xacro (robot description, xacro)
@@ -4,5 +4,5 @@
   <material name="pebble"><color rgba="0.55 0.42 0.75 1"/></material>
   <link name="base_link">
-    <inertial><origin xyz="0.000000 0.000000 0.024500"/><mass value="1.4398"/><inertia ixx="4.058e-03" ixy="0" ixz="0" iyy="4.058e-03" iyz="0" izz="7.600e-03"/></inertial>
+    <inertial><origin xyz="-0.002120 -0.003950 -0.002550"/><mass value="1.5276"/><inertia ixx="4.680112e-03" ixy="-9.017100e-05" ixz="-1.524260e-04" iyy="5.389033e-03" iyz="-2.022110e-04" izz="6.680401e-03"/></inertial>
     <visual><origin xyz="0 0 0.018"/>
       <geometry><cylinder radius="0.1100" length="0.024"/></geometry>
@@ -15,4 +15,14 @@
     <collision><origin xyz="0 0 0.044"/>
       <geometry><cylinder radius="0.0770" length="0.028"/></geometry></collision>
+    <visual name="belly_tub"><origin xyz="0.00220 -0.02000 -0.03670"/>
+      <geometry><box size="0.19940 0.05480 0.03740"/></geometry>
+      <material name="pebble"/></visual>
+    <collision name="belly_tub"><origin xyz="0.00220 -0.02000 -0.03670"/>
+      <geometry><box size="0.19940 0.05480 0.03740"/></geometry></collision>
+    <visual name="belly_shelf"><origin xyz="0.00000 0.04160 -0.03220"/>
+      <geometry><box size="0.11400 0.05880 0.04440"/></geometry>
+      <material name="pebble"/></visual>
+    <collision name="belly_shelf"><origin xyz="0.00000 0.04160 -0.03220"/>
+      <geometry><box size="0.11400 0.05880 0.04440"/></geometry></collision>
   </link>
   <xacro:macro name="pebble_leg" params="i angle">

Commit message: 9q wip 3: integration - latch + wiring merged, the CAD tree green, the sim on real masses
Merges build/wf3-latch (cec4b15: the tray's I3 strike slotted along the slide, the
tray comes out) and build/wf3-wiring (80cebbb: the bay / shelf / stand requests
closed, the retired parts gone everywhere), then closes their requests to each
other and runs the whole pipeline on one tree.

CAD
- part_busboard reads the adapter's holes and the buck's cap_l from
  part_avionics.BOARDS (the one copy, B108); its ADAPTER_HOLES / BUCK_CAP_L copies go.
- part_deck: the grid-hole job text names the hub shelf, not the star-board bracket.
- make_viewer: tray_latch_boss in the body row.
- run_all_checks: 30/30 modules, check_printability 61 parts PLATE CLEAN; the four
  body-layout parts and tray_latch_boss exported for the first time.
- fem_check: the coxa_yaw_base case pinned the WHOLE underside, the 0.2-relieved face
  included. It is now held by the docked I1 support (B118): the inboard pads (x <=
  seat_relief_x0 over the deck), the two seat flanks, the two thumbscrew heads in
  tension, each case by what bears in it (V: pads + screws, the seats lift +0.04..+0.36
  in the FEM; R-: seats + screws; L+/L-: the pressing side's pads, both seats, the
  lifting side's screw). Result: coxa_yaw_base FAILS, SF 1.10 in V (von Mises 30.4 MPa
  p99.9, peak at the vee socket (-33.1, -16.1, -1.4), cup deflection 2.29); with the
  old grip it read 3.32 (2.93 recorded). A measured finding for the owner, not fixed.
- --derived: preview, estimate, drawings (FreeCAD ran: 10/10 sheets current), the print
  pack (49 pages, carries the FEM FAIL), the viewer and the assembly views rebuilt.

Sim (pick 13, the D064 belly)
- rocky_model.belly_boxes(): the shelf is its PLATE box (params x / y, bottom_z to the
  deck), plus belly_posts(): three Ø14 post columns (plate underside to the deck);
  belly_geom_names() for the contact reports. The one hull box (grown north to y 71 by
  the (26, 64) pad) was where leg 0 touched in 20/20 recover1 falls; now recover1 x 40
  seeds under the supervisor: stood 39/40, belly contacts 2/40 falls, legs 1/4, in
  NORMAL only (the drop fixture), none on the shelf.
- build_mjcf / generate_urdf write the posts as cylinders and the belly at 1 um (the
  plate's -1.125 centre).
- mass_audit on the real STLs (no --allow-missing): tray resting at TRAY_Z 5.1, the
  tray_latch_boss weighed under the tongue, the sled's rest lift 2.10 (part_bay), the
  bay parts at PETG. Torso 1555.2 g at (-2.21, -4.63, -3.17) (was 1439.8 g at z 24.5
  on the cylinders; 1527.6 provisional); robot 2843.2 g.
- Fingerprint 87215110e9c4 -> deae868522cc (provisional c10b970d2bb2); every RL
  checkpoint is legacy on it.
- torque_audit: self-right knee 1.46 N m, 49.5 % of ST3215 (WARM).
- tests: test_belly follows the plate box + posts; the feasibility test folds leg 0 at
  hip -70 (-65 met only the old hull).

Co-Authored-By: Claude Opus 5.5 <noreply@anthropic.com>
Claude-Session: https://claude.ai/code/session_01XWxNpsfCHorgwmudjicXmk

File: ros2/rocky_description/urdf/pebble.urdf (robot description, URDF)
Before this commit: robot pebble, 26 links, 25 joints
Links:
- link base_link: mass 1.5276 -> 1.5552; geometry collision box size=0.110150 0.052100 0.044400; collision box size=0.197400 0.054800 0.037400

File: ros2/rocky_description/urdf/pebble.urdf.xacro (robot description, xacro)
@@ -4,5 +4,5 @@
   <material name="pebble"><color rgba="0.55 0.42 0.75 1"/></material>
   <link name="base_link">
-    <inertial><origin xyz="-0.002120 -0.003950 -0.002550"/><mass value="1.5276"/><inertia ixx="4.680112e-03" ixy="-9.017100e-05" ixz="-1.524260e-04" iyy="5.389033e-03" iyz="-2.022110e-04" izz="6.680401e-03"/></inertial>
+    <inertial><origin xyz="-0.002210 -0.004630 -0.003170"/><mass value="1.5552"/><inertia ixx="4.727840e-03" ixy="-9.472400e-05" ixz="-1.577160e-04" iyy="5.546485e-03" iyz="-2.393050e-04" izz="6.802222e-03"/></inertial>
     <visual><origin xyz="0 0 0.018"/>
       <geometry><cylinder radius="0.1100" length="0.024"/></geometry>
@@ -15,14 +15,29 @@
     <collision><origin xyz="0 0 0.044"/>
       <geometry><cylinder radius="0.0770" length="0.028"/></geometry></collision>
-    <visual name="belly_tub"><origin xyz="0.00220 -0.02000 -0.03670"/>
-      <geometry><box size="0.19940 0.05480 0.03740"/></geometry>
+    <visual name="belly_tub"><origin xyz="0.001200 -0.020000 -0.036700"/>
+      <geometry><box size="0.197400 0.054800 0.037400"/></geometry>
       <material name="pebble"/></visual>
-    <collision name="belly_tub"><origin xyz="0.00220 -0.02000 -0.03670"/>
-      <geometry><box size="0.19940 0.05480 0.03740"/></geometry></collision>
-    <visual name="belly_shelf"><origin xyz="0.00000 0.04160 -0.03220"/>
-      <geometry><box size="0.11400 0.05880 0.04440"/></geometry>
+    <collision name="belly_tub"><origin xyz="0.001200 -0.020000 -0.036700"/>
+      <geometry><box size="0.197400 0.054800 0.037400"/></geometry></collision>
+    <visual name="belly_shelf"><origin xyz="-0.001125 0.038250 -0.032200"/>
+      <geometry><box size="0.110150 0.052100 0.044400"/></geometry>
       <material name="pebble"/></visual>
-    <collision name="belly_shelf"><origin xyz="0.00000 0.04160 -0.03220"/>
-      <geometry><box size="0.11400 0.05880 0.04440"/></geometry></collision>
+    <collision name="belly_shelf"><origin xyz="-0.001125 0.038250 -0.032200"/>
+      <geometry><box size="0.110150 0.052100 0.044400"/></geometry></collision>
+    <visual name="belly_shelf_post0"><origin xyz="-0.050000 0.034000 -0.024650"/>
+      <geometry><cylinder radius="0.007000" length="0.029300"/></geometry>
+      <material name="pebble"/></visual>
+    <collision name="belly_shelf_post0"><origin xyz="-0.050000 0.034000 -0.024650"/>
+      <geometry><cylinder radius="0.007000" length="0.029300"/></geometry></collision>
+    <visual name="belly_shelf_post1"><origin xyz="0.050000 0.034000 -0.024650"/>
+      <geometry><cylinder radius="0.007000" length="0.029300"/></geometry>
+      <material name="pebble"/></visual>
+    <collision name="belly_shelf_post1"><origin xyz="0.050000 0.034000 -0.024650"/>
+      <geometry><cylinder radius="0.007000" length="0.029300"/></geometry></collision>
+    <visual name="belly_shelf_post2"><origin xyz="0.026000 0.064000 -0.024650"/>
+      <geometry><cylinder radius="0.007000" length="0.029300"/></geometry>
+      <material name="pebble"/></visual>
+    <collision name="belly_shelf_post2"><origin xyz="0.026000 0.064000 -0.024650"/>
+      <geometry><cylinder radius="0.007000" length="0.029300"/></geometry></collision>
   </link>
   <xacro:macro name="pebble_leg" params="i angle">
