Commit message: 9q wip 4: review fixes - shell vs docked base, tray release with the carapace, sim mirrors checked, belly-free drops, resume contract
Blockers
- part_shell: every docked coxa_yaw_base cut 42.80 mm^3 into its sector (the cup's back
  wall, leg x -38.5 = body r 71.5, stood 0.5 inside the leg arch's x 72; on main too).
  cup_back_relief() takes the sector FIT off the wall's back, sides and top, over the
  wall's width only (x 71.2..73, |y| <= 9.8, z -0.3..45.5): moving the whole arch in to
  71.2 would also cut the latch pad and the feet (its |y| <= 40 profile). keepouts() now
  holds the real station-posed base + yaw servo, gated at 0 mm^3, and the sector-to-base
  gap is gated >= FIT: 0.00 / 0.00 mm^3, 0.30 mm. Sector 25385.9 -> 25316.6 mm^3 (STL).
  Torso 1555.2 -> 1555.0 g at (-2.21, -4.63, -3.18); robot 2843.0 g; fingerprint
  deae868522cc -> c3e82f13b671 (mass_audit -> build_mjcf -> URDF -> parity OK ->
  torque_audit: knee 1.46 N m, 50 % WARM, unchanged).
- part_avionics: _vol no longer swallows exceptions (872dba5); an OCCT failure fails
  the module instead of reading 0 mm^3.

Majors
- part_avionics: the release path with the carapace ON is a reported row: sector 2 at
  slide 14 (4.04 mm^3), its I3 cartridge by 16 (5.34), sector 3 at lift 10 (0.34),
  sector 4 by 14, the cap by 18, sector 1 by 42; sector 0 never (the reviewer's 2, 3, 4 +
  cap is the straight lift to 18; to 45 it meets sector 1 too). The gated path says
  "carapace off"; the module doc says the carapace comes off first (with the robot off
  the stand and the sled out: the strike's driver column).
- gen_print_pack / print_estimate: the tray rows say how it comes out (carapace off,
  off the stand, sled out, OPEN, slide 16 south, the slot stops it at 16.5, lift) and
  the boss's LATCH_WALL 1.6; the stale "cannot slide out until the slotted strike is
  cut" and "0.85 of wall: VERIFY" are gone. PRINT_PREP_PACK.pdf regenerated (--derived).
- ci.yml: the cad-job filter takes gait/rocky_model.py, sim/mass_budget.json and
  gait/pebble_gait.py.
- mass_audit: TRAY_REST_DROP and RAIL_POSE_X derive from params.clearance_fit;
  tray_plate_z() / sled_z() / yaw_case_leg() expose the poses. New
  cad/check_sim_mirror.py (run_all_checks POST, so the cad job) asserts every pose-table
  mirror against its part module (part_avionics SEAT_Z / TRAY_Z / BOSS_H / TONGUE_Y /
  RAIL_POSE_X / PI_BOARD_DX, part_bay SLED_Z0 - ZF, part_battery SLED_T, leg_frame
  HUB_Z1 / ZC_YAW, part_busboard SHELF_BOARDS), rocky_model's belly against iface /
  part_busboard, and the exported bay_tub / hub_shelf against the sim's boxes:
  bay_tub 0 vertices outside the box + iface.BAY_TUB_OUTSIDE (the documented
  protrusions, now a table); hub_shelf at most 0.60 past the plate box + post columns
  (the plate's NOTCH_R fillets; gated at 1.0).
- params interfaces.hub_shelf.pad_d 14: part_busboard's pads and rocky_model's post
  columns read the one key (SHELF_PAD_WALL_MM gone; same Ø14 today).
- RecoverEnv drop_clear_of_belly (default True, in config()): a drop's joint draw that
  starts a leg inside a belly geom is drawn again (3.7 % of draws; 15/400 seeds); a kept
  draw lands exactly as before (mj_fwdPosition only). eval_recover.env_for replays a
  contract without the key on the old stream. Test: 60 seeds never start in the belly.
- train_ppo: --hip-clamp params|none|DEG and --belly-drops reach the env; a resume whose
  action map differs (rl_common.action_map_mismatch: hip floor / its legs) is refused
  (a pre-D064 checkpoint continues with --hip-clamp none). Tests.

Test re-pinned
- test_playground_guards: the chaotic wave + push fall used 65 N, the band's edge: on
  deae868522cc 60-65 N land it at 164.8 deg (55-58 and 66-80 tip it to 150-155 and the
  keel rolls it back), on c3e82f13b671 60-64. 62 N, the middle of both.

Minors
- params comments (lug_release south only + carapace; standoff_h's K3 sentence),
  RIGHTER_CLAMP_LEGS literal gone (params is the one copy; a floor with no legs raises),
  part_deck counts a PENDING audit row as a failure, part_bay gates the flexure webs'
  stress (23.4 < 35 MPa) and the hook tab's strain (1.17 < 2.33 %), the busboard tub
  label 1.92 (riser clip), the fallback masses in one place (rocky_model.FALLBACK_MASS_G;
  generate_urdf warns), test_belly asserts the committed budget is not provisional,
  .claude/worktrees ignored + ruff extend-exclude, stale docstrings (recover env belly,
  part_shell deck v0.5, mass_audit CoM, CI / run_all_checks timings).

Checks: run_all_checks --derived 37/37 TREE CLEAN (check_printability 61 parts, the new
check_sim_mirror CLEAN; derived: preview, estimate, 10/10 drawings current, the print
pack 49 pages, viewer, 13 assembly views); pytest sim/tests 819 passed + the re-pinned
one (42 passed in its file), driver/gait/harness 305 passed, harness slow 2 passed;
run_sim walk 189 mm, turn 41.7 deg; ruff clean; TOOLS.md current.

Co-Authored-By: Claude Fable 5.1 <noreply@anthropic.com>
Claude-Session: https://claude.ai/code/session_01XWxNpsfCHorgwmudjicXmk

File: ros2/rocky_description/urdf/pebble.urdf (robot description, URDF)
Before this commit: robot pebble, 26 links, 25 joints
Links:
- link base_link: mass 1.5552 -> 1.5550

File: ros2/rocky_description/urdf/pebble.urdf.xacro (robot description, xacro)
@@ -4,5 +4,5 @@
   <material name="pebble"><color rgba="0.55 0.42 0.75 1"/></material>
   <link name="base_link">
-    <inertial><origin xyz="-0.002210 -0.004630 -0.003170"/><mass value="1.5552"/><inertia ixx="4.727840e-03" ixy="-9.472400e-05" ixz="-1.577160e-04" iyy="5.546485e-03" iyz="-2.393050e-04" izz="6.802222e-03"/></inertial>
+    <inertial><origin xyz="-0.002210 -0.004630 -0.003180"/><mass value="1.5550"/><inertia ixx="4.726674e-03" ixy="-9.472200e-05" ixz="-1.576910e-04" iyy="5.545323e-03" iyz="-2.392530e-04" izz="6.800853e-03"/></inertial>
     <visual><origin xyz="0 0 0.018"/>
       <geometry><cylinder radius="0.1100" length="0.024"/></geometry>
