Commit message: 9q: the body layout built from the owner's 15 picks (D064) - the docs, the buy-and-print order, the code map, the tray tab holes
Documentation for the D064 build, after the five build workflows (d99cdc2 the I1 seats fix and
the foundation; a82f8ad the six parts; ef7c923 integration; 3ec6ab5 review fixes; c0947bf the
re-run records):
- INTERFACES I1 (seats as built, the stance load path, the FEM finding), I3 (the slide-slot
  strike), I4 and I5 revised (decision 11); WIRING_HARNESS under the deck (shelf, lanes, the
  14 AWG route, the (0, 50) slot, UART for the bus adapter, one USB-A); SERVO_NOTES numbers.
- BOM: B-24 = the 30.5 x 30.5 PDB; new B-25..B-30, C-05, X-20 (the carrier's female XT60,
  M3 x 30 shelf posts, ISO 7380 tabs, spacers, the foam pad, the UART lead, the right-angle
  USB-A, the long driver); core robot $1,265. bom/README totals.
- PRINT_PLAN (batch 0 = the port coupons + the fit ladder; the hold on coxa_yaw_base x5),
  ASSEMBLY_GUIDE (the body as built, trimmed), docs/BUY_AND_PRINT_ORDER.md (NEW: eleven steps
  in spend order with costs, grams, hours and gates), docs/CODE_MAP.md (NEW: the directory map,
  the data flow and fifteen how-do-I recipes with file:function pointers).
- DESIGN_BACKLOG: 20 rows closed, B139-B155 added (the coxa base stall case SF 1.10 is the
  owner's next decision); decisions D064; BUILD_LOG 9q; README status; SIM_GUIDE / RL_GUIDE /
  COCKPIT_GUIDE / DESIGN_CHANGE_GUIDE updated; sim/experiments/README re-recorded.
- Pruned: BODY_LAYOUT_PROPOSAL, REVIEW_2026-09-22, PERCEPTION_PLAN and BUILD_LOG sessions
  8e-9k moved to docs/archive/; ROBOT_AS_DATA + SCALE_UP_NOTES merged into DESIGN_CHANGE_GUIDE;
  PLACES condensed. Live docs 9.6k -> about 7k lines.
- One CAD fix found by the docs critic (B155): the tray's two north tab holes at (+-40, 20) are
  thread-forming Ø2.8 again (nothing under them to thread into); deck re-exported, derived
  outputs rebuilt, masses unchanged at 0.1 g, fingerprint c3e82f13b671 -> 965f4f70e5d1 (the
  torso inertia's 8th decimal). CAD 31/31, --derived 37/37, sim 820 passed.

Co-Authored-By: Claude Fable 5.1 <noreply@anthropic.com>
Claude-Session: https://claude.ai/code/session_01XWxNpsfCHorgwmudjicXmk

File: ros2/rocky_description/urdf/pebble.urdf.xacro (robot description, xacro)
@@ -4,5 +4,5 @@
   <material name="pebble"><color rgba="0.55 0.42 0.75 1"/></material>
   <link name="base_link">
-    <inertial><origin xyz="-0.002210 -0.004630 -0.003180"/><mass value="1.5550"/><inertia ixx="4.726674e-03" ixy="-9.472200e-05" ixz="-1.576910e-04" iyy="5.545323e-03" iyz="-2.392530e-04" izz="6.800853e-03"/></inertial>
+    <inertial><origin xyz="-0.002210 -0.004630 -0.003180"/><mass value="1.5550"/><inertia ixx="4.726687e-03" ixy="-9.472300e-05" ixz="-1.576910e-04" iyy="5.545358e-03" iyz="-2.392510e-04" izz="6.800901e-03"/></inertial>
     <visual><origin xyz="0 0 0.018"/>
       <geometry><cylinder radius="0.1100" length="0.024"/></geometry>
